Commit message: Improved position of retargeting frames on fingertips of sharpa urdf to better match DITTO fingerpads.

File: retargeting_teleop/retargeting/assets/sharpa_right/right_sharpa_wave.urdf (robot description, URDF)
Before this commit: robot right_sharpa_wave, 36 links, 35 joints
Joints:
- joint right_index_retargeting_pad_joint: origin xyz=0 0 0 rpy=3.141592653589793 -1.5707963267949 0 -> xyz=0.0 0 -0.01 rpy=3.141592653589793 -1.5707963267949 0
- joint right_thumb_MCP_FE: limit lower=-0.35 upper=1.3963 effort=1.864 velocity=16.07692878 -> lower=-0.1 upper=1.3963 effort=1.864 velocity=16.07692878
- joint right_thumb_retargeting_pad_joint: origin xyz=0 0 0 rpy=3.141592653589793 -1.5707963267949 0 -> xyz=0.0 0 -0.010 rpy=3.141592653589793 -1.5707963267949 0
