Commit message: Adding ditto_3f urdf for 3 finger leader exo. Adapting sharpa urdf to include middle finger retargeting pad.

File: retargeting_teleop/retargeting/assets/sharpa_right/right_sharpa_wave.urdf (robot description, URDF)
Before this commit: robot right_sharpa_wave, 36 links, 35 joints
Links:
- added link right_middle_retargeting_pad, mass 1.0E-06
Joints:
- added joint right_middle_retargeting_pad_joint: type fixed, parent right_middle_fingertip, child right_middle_retargeting_pad, origin xyz=0.0 0 -0.01 rpy=3.141592653589793 -1.5707963267949 0
