Commit message: Support of new ditto_3f_v2 leader hardware. Decent config tunning in ditto_3f_mixed_sources_tune.yaml

File: retargeting_teleop/retargeting/assets/ditto_3f_leader_v2/ditto_3f_leader_v2.urdf (robot description, URDF)
Before this commit: robot ditto_leader_urdf_assembly, 11 links, 10 joints
Links:
- added link middle_fingerpad, mass 0.00332341020047785; collision mesh filename=meshes/middle_fingerpad.STL; visual mesh filename=meshes/middle_fingerpad.STL
- added link middle_link_0, mass 0.0268394050979217; collision mesh filename=meshes/middle_link_0.STL; visual mesh filename=meshes/middle_link_0.STL
- added link middle_link_1, mass 0.0329000270028115; collision mesh filename=meshes/middle_link_1.STL; visual mesh filename=meshes/middle_link_1.STL
- added link middle_link_2, mass 0.00252674876938612; collision mesh filename=meshes/middle_link_2.STL; visual mesh filename=meshes/middle_link_2.STL
- link base_link: mass 0.0870719662910429 -> 0.104263737833624
- link index_fingerpad: mass 0.00293503442151317 -> 0.00293503442078025
- link index_link_2: mass 0.00252674876938613 -> 0.00252674876938614
- link thumb_fingerpad: mass 0.00282848549611835 -> 0.00282848549611836
Joints:
- added joint middle_fingerpad_joint: type fixed, parent middle_link_2, child middle_fingerpad, origin xyz=0.0302000000000001 0.00700000000000259 0.0669999999999999 rpy=-1.5707963267949 0 0, axis 0 0 0
- added joint middle_joint_0: type revolute, parent base_link, child middle_link_0, origin xyz=-0.025 0 0 rpy=0 0 -3.1416, axis 0 0 1, limit lower=-0.3 upper=0.3 effort=0 velocity=0
- added joint middle_joint_1: type revolute, parent middle_link_0, child middle_link_1, origin xyz=0.067 0 0.046 rpy=1.5708 0 -1.5708, axis 0 0 1, limit lower=-0.17 upper=1.57 effort=0 velocity=0
- added joint middle_joint_2: type revolute, parent middle_link_1, child middle_link_2, origin xyz=0.0485 0 0 rpy=0 0 0, axis 0 0 1, limit lower=-0.1 upper=1.57 effort=0 velocity=0
- joint index_joint_1: origin xyz=0.03 0 0.046 rpy=1.5707963267949 0 1.57079632679489 -> xyz=0.03 0 0.046 rpy=1.5708 0 1.5708
- joint index_joint_2: origin xyz=0.0409999999999936 0 0 rpy=0 0 0 -> xyz=0.041 0 0 rpy=0 0 0
- joint thumb_fingerpad_joint: origin xyz=0.0340000000000001 -0.00500000000000015 -0.0398000000000016 rpy=1.80666825946075 -0.379498136323909 0.503100653479423 -> xyz=0.034 -0.00499999999999983 -0.0398000000000015 rpy=1.80666825946076 -0.379498136323909 0.503100653479423
- joint thumb_joint_0: axis 0 -0.16711 0.98594 -> 0 0 1; origin xyz=-0.0021417 -0.080436 0.0054795 rpy=0.016838 -0.18167 -1.6637 -> xyz=-0.00081039 -0.081987 -0.0022549 rpy=0.18474 -0.18167 -1.6637
- joint thumb_joint_1: origin xyz=0.033941 0.023014 0.067326 rpy=1.4005 -0.79917 2.4717 -> xyz=0.033941 0.033941 0.070534 rpy=1.5708 -0.68717 2.3562
- joint thumb_joint_2: origin xyz=0.0592471988937204 0.0378393192831767 -0.019789507993749 rpy=1.14448873095508 0.194946179240087 1.71050085923731 -> xyz=0.059247 0.037839 -0.01979 rpy=1.1445 0.19495 1.7105

File: retargeting_teleop/retargeting/assets/sharpa_right/right_sharpa_wave.urdf (robot description, URDF)
Before this commit: robot right_sharpa_wave, 37 links, 36 joints
Joints:
- joint right_index_retargeting_pad_joint: origin xyz=0.0 0 -0.01 rpy=3.141592653589793 -1.5707963267949 0 -> xyz=-0.005 0 -0.01 rpy=3.141592653589793 -1.5707963267949 0
- joint right_middle_retargeting_pad_joint: origin xyz=0.0 0 -0.01 rpy=3.141592653589793 -1.5707963267949 0 -> xyz=-0.005 0 -0.01 rpy=3.141592653589793 -1.5707963267949 0
- joint right_thumb_retargeting_pad_joint: origin xyz=0.0 0 -0.010 rpy=3.141592653589793 -1.5707963267949 0 -> xyz=-0.005 0 -0.010 rpy=3.141592653589793 -1.5707963267949 0
