Commit message: Consolidating use of 2f and 3f urdfs. Adding visualizer for debugging force sensing sources from sharpa hand in view_force_sensing.py.

File: retargeting_teleop/retargeting/assets/ditto_3f_leader/ditto_3f_leader.urdf (robot description, URDF)
Before this commit: robot ditto_3f_leader, 15 links, 14 joints
Links:
- link base_link: mass 0.109125547143221 -> 0.104263737833624
- link index_fingerpad: mass 0.00293503442078024 -> 0.00293503442078025
- link index_link_2: mass 0.00252674876938613 -> 0.00252674876938614
- link middle_fingerpad: mass 0.00354844692145956 -> 0.00332341020047785
- link middle_link_0: mass 0.0257036203076206 -> 0.0268394050979217
- link middle_link_2: mass 0.00252674876938613 -> 0.00252674876938612
- link thumb_link_1: mass 0.0337789978005482 -> 0.0337789978005483
- link thumb_link_3: mass 0.00252674889330346 -> 0.00252674889330345
Joints:
- joint index_joint_0: axis 0 0 -1 -> 0 0 1; limit lower=-0.8 upper=0.3 effort=0 velocity=0 -> lower=-0.3 upper=0.8 effort=0 velocity=0
- joint index_joint_1: axis 0 0 -1 -> 0 0 1; limit lower=-1.57 upper=0.17 effort=0 velocity=0 -> lower=-0.17 upper=1.57 effort=0 velocity=0; origin xyz=0.03 0 0.046 rpy=1.5707963267949 0 1.57079632679489 -> xyz=0.03 0 0.046 rpy=1.5708 0 1.5708
- joint index_joint_2: axis 0 0 -1 -> 0 0 1; limit lower=-1.57 upper=0.1 effort=0 velocity=0 -> lower=-0.1 upper=1.57 effort=0 velocity=0; origin xyz=0.0409999999999935 0 0 rpy=0 0 0 -> xyz=0.041 0 0 rpy=0 0 0
- joint middle_fingerpad_joint: origin xyz=0.0302000000000001 0.00975000000000249 0.0702999999999999 rpy=-1.5707963267949 0 0 -> xyz=0.0302000000000001 0.00700000000000259 0.0669999999999999 rpy=-1.5707963267949 0 0
- joint middle_joint_0: axis 0 0 -1 -> 0 0 1; origin xyz=-0.0395 0.0005 0 rpy=0 0 3.1416 -> xyz=-0.025 0 0 rpy=0 0 -3.1416
- joint middle_joint_1: axis 0 0 -1 -> 0 0 1; limit lower=-1.57 upper=0.17 effort=0 velocity=0 -> lower=-0.17 upper=1.57 effort=0 velocity=0; origin xyz=0.052 0 0.046 rpy=1.5708 0 -1.5708 -> xyz=0.067 0 0.046 rpy=1.5708 0 -1.5708
- joint middle_joint_2: axis 0 0 -1 -> 0 0 1; limit lower=-1.57 upper=0.1 effort=0 velocity=0 -> lower=-0.1 upper=1.57 effort=0 velocity=0
- joint thumb_fingerpad_joint: origin xyz=0.034 -0.00499999999999969 -0.0398 rpy=1.80666825946076 -0.379498136323909 0.503100653479423 -> xyz=0.034 -0.00499999999999983 -0.0398000000000015 rpy=1.80666825946076 -0.379498136323909 0.503100653479423
- joint thumb_joint_0: axis 0 -0.167114290573186 0.985937530417734 -> 0 0 1; origin xyz=-0.00214172528372005 -0.0804363017815774 0.00547954198946005 rpy=0.016838154197939 -0.181665966850915 -1.66373584590886 -> xyz=-0.00081039 -0.081987 -0.0022549 rpy=0.18474 -0.18167 -1.6637
- joint thumb_joint_1: origin xyz=0.0339411254969603 0.023013567589507 0.0673262918632758 rpy=1.40051047580421 -0.799169731618551 2.47174579176664 -> xyz=0.033941 0.033941 0.070534 rpy=1.5708 -0.68717 2.3562
- joint thumb_joint_2: origin xyz=0.0592471988937203 0.0378393192831765 -0.0197895079937487 rpy=1.14448873095508 0.194946179240088 1.71050085923731 -> xyz=0.059247 0.037839 -0.01979 rpy=1.1445 0.19495 1.7105
